File: MCU_Proto/MCU_Prototype/MCU_Prototype.kicad_pcb (KiCad board)
At the start: 2 copper layers, 85 x 70 mm, 30 parts, among them J1 UART, J3 SWD, J4 USB_A, J5 PIN1-PIN16, J6 PIN17-PIN32, J7 PIN33-PIN48, J8 PIN49-PIN64, SW1 SW_DPDT_x2, SW2 SW_Push, U1 LD1117S33CTR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

Commit message: Routed VDD and GND
Routing:
- net VDD: track 45.7 -> 88.2 mm, vias 0 -> 6
- net GND: track 0.00 -> 21.2 mm, vias 0 -> 3
- net NRST: track 106.0 -> 106.8 mm
- added copper zone on In1.Cu, net VDD
Other:
- copper layers 2 -> 4
