File: MCU_Prototype/MCU_Prototype.kicad_pcb (KiCad board)
At the start: 4 copper layers, 71.5 x 69.5 mm, 35 parts, among them J1 UART, J2 Battery, J3 SWD, J4 USB_A, J5 PIN1-PIN16, J6 PIN17-PIN32, J7 PIN33-PIN48, J8 PIN49-PIN64, SW1 SW_DPDT_x2, SW2 SW_Push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

Commit message: Added silkscreen
Parts:
- removed C14: 4.7u, Capacitor_THT:CP_Radial_D5.0mm_P2.00mm
- removed C4: 100n, Capacitor_SMD:C_0805_2012Metric
Routing:
- net VDD: track 86.3 -> 80.6 mm, vias 6 -> 5
- net GND: track 20.7 -> 16.7 mm, vias 93 -> 95
- net PC_13: track 20.5 -> 20.0 mm
Other:
- board text added: "Version 1.0 2022-10-14 Project course E7032E Johan Axenhag"
